Commit message: feat: switch core simulation engine to PyBullet Headless with native motor control and LiDAR raycasting

File: robot.urdf (robot description, URDF)
Before this commit: robot cmodel_agv, 8 links, 7 joints
Links:
- added link front_caster_link, mass 1.0; collision sphere radius=0.05
- added link rear_caster_link, mass 1.0; collision sphere radius=0.05
- link base_footprint: mass None -> 0.001
- link imu_link: mass None -> 0.05
- link laser0_link: mass None -> 0.1
- link laser1_link: mass None -> 0.1
- link laser_link: mass None -> 0.1
- link left_wheel_link: mass None -> 4.0; geometry collision cylinder length=0.0500 radius=0.1150; visual cylinder length=0.0500 radius=0.1150
- link right_wheel_link: mass None -> 4.0; geometry collision cylinder length=0.0500 radius=0.1150; visual cylinder length=0.0500 radius=0.1150
Joints:
- added joint front_caster_joint: type fixed, parent base_link, child front_caster_link, origin xyz=0.8000 0 0.0500 rpy=0 0 0
- added joint rear_caster_joint: type fixed, parent base_link, child rear_caster_link, origin xyz=-0.2000 0 0.0500 rpy=0 0 0
